File: sketch/sigma-computer/ALU.sch (KiCad schematic (older format))
At the start: 8 parts

Commit message: Started the microcode compiler
Parts:
- added U? (x2): 74HCT244, symbol 74xx:74HCT244
- added U? (x2): 74HCT240, symbol 74xx:74HCT240
Connections:
- wire segments 295 -> 392
