File: sketch/sigma-computer/ALU.sch (KiCad schematic (older format))
At the start: 8 parts

Commit message: Changes in the schematic
Parts:
- removed U? (x2): 74HCT244, symbol 74xx:74HCT244
- removed U? (x2): 74HCT374, symbol 74xx:74HCT374
- removed U? (x4): 74HC283, symbol Additional74:74HC283
- added U? (x4): 74HC283, symbol Additional74:74HC283
- added U?: 74LCX16244, symbol Additional74:74LCX16244
Connections:
- net labels added: Clock, E_HIGH_IN
- wire segments 164 -> 76
Other:
- note added: "Register E"
- note removed: "Register IAR"
