File: sketch/sigma-computer/BIOS.sch (KiCad schematic (older format))
At the start: 2 parts

Commit message: Changes in ID
Connections:
- wire segments 32 -> 64
Changed lines of the file:
@@
 $EndComp
 Wire Wire Line
-	11150 6500 11150 500
+	11100 500  11100 4400
 Wire Wire Line
-	11200 500  11200 6500
+	11050 6500 11050 4300
 Wire Wire Line
-	11100 500  11100 6500
+	11000 6500 11000 4200
 Wire Wire Line
-	11050 6500 11050 500
+	10950 500  10950 4100
 Wire Wire Line
-	11000 6500 11000 500
-Wire Wire Line
-	10950 500  10950 6500
-Wire Wire Line
-	10900 500  10900 6500
-Wire Wire Line
-	10850 6500 10850 500
+	10900 500  10900 4000
 Wire Wire Line
 	10750 6500 10750 1700
@@
 	1    0    0    -1
 $EndComp
+Wire Wire Line
+	11150 6500 11150 4500
+Wire Wire Line
+	11200 500  11200 4600
+Wire Wire Line
+	10850 6500 10850 3900
+Wire Wire Line
+	8800 4600 11200 4600
+Connection ~ 11200 4600
+Wire Wire Line
+	11200 4600 11200 6500
+Wire Wire Line
+	8800 4500 11150 4500
+Connection ~ 11150 4500
+Wire Wire Line
+	11150 4500 11150 500
+Wire Wire Line
+	8800 4400 11100 4400
+Connection ~ 11100 4400
+Wire Wire Line
+	11100 4400 11100 6500
+Wire Wire Line
+	8800 4300 11050 4300
+Connection ~ 11050 4300
+Wire Wire Line
+	11050 4300 11050 500
+Wire Wire Line
+	8800 4200 11000 4200
+Connection ~ 11000 4200
+Wire Wire Line
+	11000 4200 11000 500
+Wire Wire Line
+	8800 4100 10950 4100
+Connection ~ 10950 4100
+Wire Wire Line
+	10950 4100 10950 6500
+Wire Wire Line
+	8800 4000 10900 4000
+Connection ~ 10900 4000
+Wire Wire Line
+	10900 4000 10900 6500
+Wire Wire Line
+	8800 3900 10850 3900
+Connection ~ 10850 3900
+Wire Wire Line
+	10850 3900 10850 500
+Wire Wire Line
+	1200 6500 1200 500
+Wire Wire Line
+	1250 500  1250 6500
+Wire Wire Line
+	1150 500  1150 6500
+Wire Wire Line
+	1100 6500 1100 500
+Wire Wire Line
+	1050 6500 1050 500
+Wire Wire Line
+	1000 500  1000 6500
+Wire Wire Line
+	950  500  950  6500
+Wire Wire Line
+	900  6500 900  500
+Wire Wire Line
+	800  6500 800  500
+Wire Wire Line
+	850  500  850  6500
+Wire Wire Line
+	750  500  750  6500
+Wire Wire Line
+	700  6500 700  500
+Wire Wire Line
+	650  6500 650  500
+Wire Wire Line
+	600  500  600  6500
+Wire Wire Line
+	550  500  550  6500
+Wire Wire Line
+	500  6500 500  500
 $EndSCHEMATC

Commit message: Changes in the schematic
Parts:
- gave numbers to parts that had none: 2
Changed lines of the file:
@@
 $Descr A4 11693 8268
 encoding utf-8
-Sheet 10 11
+Sheet 10 10
 Title ""
 Date ""
@@
 $EndDescr
 $Comp
-L Memory_Flash:SST39SF010 U?
+L Memory_Flash:SST39SF010 U53
 U 1 1 5D29CFD9
 P 8200 2300
-F 0 "U?" H 8200 3781 50  0000 C CNN
+F 0 "U53" H 8200 3781 50  0000 C CNN
 F 1 "SST39SF010" H 8200 3690 50  0000 C CNN
 F 2 "" H 8200 2600 50  0001 C CNN
@@
 	10800 1800 10800 6500
 $Comp
-L Memory_Flash:SST39SF010 U?
+L Memory_Flash:SST39SF010 U54
 U 1 1 5D4D3771
 P 8200 5100
-F 0 "U?" H 8200 6581 50  0000 C CNN
+F 0 "U54" H 8200 6581 50  0000 C CNN
 F 1 "SST39SF010" H 8200 6490 50  0000 C CNN
 F 2 "" H 8200 5400 50  0001 C CNN
