File: sketch/sigma-computer/Registers_A-F.sch (KiCad schematic (older format))
At the start: 12 parts

Commit message: Changes in the schematic
Parts:
- gave numbers to parts that had none: 12
Connections:
- wire segments 767 -> 760
