File: sketch/sigma-computer/memory.sch (KiCad schematic (older format))
At the start: 2 parts

Commit message: Changes in the schematic
Parts:
- gave numbers to parts that had none: 2
Changed lines of the file:
@@
 $Descr A4 11693 8268
 encoding utf-8
-Sheet 6 11
+Sheet 6 10
 Title ""
 Date ""
@@
 	10450 500  10450 6500
 $Comp
-L SRAM:HM62256LP-8 U?
+L SRAM:HM62256LP-8 U39
 U 1 1 5D560ECE
 P 1950 1700
-F 0 "U?" H 1950 2325 50  0000 C CNN
+F 0 "U39" H 1950 2325 50  0000 C CNN
 F 1 "HM62256LP-8" H 1950 2234 50  0000 C CNN
 F 2 "" H 1950 650 50  0001 C CNN
@@
 $EndComp
 $Comp
-L SRAM:HM62256LP-8 U?
+L SRAM:HM62256LP-8 U40
 U 1 1 5D5628BD
 P 1950 3600
-F 0 "U?" H 1950 4225 50  0000 C CNN
+F 0 "U40" H 1950 4225 50  0000 C CNN
 F 1 "HM62256LP-8" H 1950 4134 50  0000 C CNN
 F 2 "" H 1950 2550 50  0001 C CNN
