File: sketch/sigma-computer/sigma-computer.sch (KiCad schematic (older format))
At the start: 0 parts

Commit message: Changes in the schematic
Changed lines of the file:
@@
 $Descr A4 11693 8268
 encoding utf-8
-Sheet 1 11
+Sheet 1 10
 Title ""
 Date ""
@@
 $EndDescr
 $Sheet
-S 650  1550 1050 1250
+S 650  1550 2400 1250
 U 5D32333B
-F0 "Registers_A-C" 50
-F1 "Registers_A-C.sch" 50
+F0 "Registers_A-F" 50
+F1 "Registers_A-F.sch" 50
 $EndSheet
 $Sheet
@@
 CPU
 $Sheet
-S 650  3000 2400 500
+S 650  4400 2400 500
 U 5D273310
 F0 "ALU" 50
@@
 $EndSheet
 $Sheet
-S 650  4400 2400 500
+S 650  3000 2400 500
 U 5D2739E4
 F0 "special-registers" 50
@@
 $EndSheet
 $Sheet
-S 2000 1550 1050 1250
-U 5D28F068
-F0 "Registers_D-F" 50
-F1 "Registers_D-F.sch" 50
-$EndSheet
-$Sheet

Commit message: Updated the schematics
Parts:
- added U? (x10): 74LCX16244, symbol Additional74:74LCX16244
- added U? (x9): 74LVC16374ADGG, symbol Additional74:74LVC16374ADGG
- added U? (x4): 74HC590, symbol 74HC253:74HC590
- added U? (x3): CD74HC137, symbol Additional74:CD74HC137
- added U? (x2): SST39SF010, symbol Memory_Flash:SST39SF010
- added U?: Demux1, symbol General:Demux1
- added U? (x4): 74HC283, symbol Additional74:74HC283
Connections:
- new net: U?.11 (O6), U?.38 (1D6) (x9)
- new net: U?.12 (O7), U?.37 (1D7) (x9)
- new net: U?.13 (O8), U?.36 (2D0) (x9)
- new net: U?.14 (O9), U?.35 (2D1) (x9)
- new net: U?.16 (O10), U?.33 (2D2) (x9)
- new net: U?.17 (O11), U?.32 (2D3) (x9)
- new net: U?.19 (O12), U?.30 (2D4) (x9)
- new net: U?.2 (O0), U?.47 (1D0) (x9)
- new net: U?.20 (O13), U?.29 (2D5) (x9)
- new net: U?.22 (O14), U?.27 (2D6) (x9)
- new net: U?.23 (O15), U?.26 (2D7) (x9)
- new net: U?.3 (O1), U?.46 (1D1) (x9)
- new net: U?.44 (1D2), U?.5 (O2) (x9)
- new net: U?.43 (1D3), U?.6 (O3) (x9)
- new net: U?.41 (1D4), U?.8 (O4) (x9)
- new net: U?.40 (1D5), U?.9 (O5) (x9)
- new net: U?.1 (Q1), U?.46 (I1) (x2)
- new net: U?.15 (Q0), U?.47 (I0) (x2)
- new net: U?.2 (Q2), U?.44 (I2) (x2)
- new net: U?.3 (Q3), U?.43 (I3) (x2)
- new net: U?.4 (Q4), U?.41 (I4) (x2)
- new net: U?.40 (I5), U?.5 (Q5) (x2)
- new net: U?.38 (I6), U?.6 (Q6) (x2)
- new net: U?.37 (I7), U?.7 (Q7) (x2)
- new net: U?.1 (A0), U?.20 (D6)
- new net: U?.10 (Y5), U?.11 (REG_F_LOW_IN)
- new net: U?.11 (Y4), U?.9 (REG_E_LOW_IN)
- new net: U?.12 (Y3), U?.7 (REG_D_LOW_IN)
- new net: U?.13 (Y2), U?.5 (REG_C_LOW_IN)
- new net: U?.14 (Y1), U?.3 (REG_B_LOW_IN)
- new net: U?.1 (REG_A_LOW_IN), U?.15 (Y0)
- new net: U?.2 (A1), U?.21 (D7)
- new net: U?.13 (D0), U?.3 (A2)
- new net: U?.15 (D2), U?.6 (OE0), U?.6 (OE0)
- new net: U?.15 (I_REG_ADDR_IN), U?.7 (Y7)
- new net: U?.13 (I_REG_OPCODE_IN), U?.9 (Y6)
- new net: U?.1 (A0), U?.17 (D3)
- new net: U?.10 (Y5), U?.12 (REG_F_LOW_OUT)
- new net: U?.10 (REG_E_LOW_OUT), U?.11 (Y4)
- new net: U?.12 (Y3), U?.8 (REG_D_LOW_OUT)
- new net: U?.13 (Y2), U?.6 (REG_C_LOW_OUT)
- new net: U?.14 (Y1), U?.4 (REG_B_LOW_OUT)
- new net: U?.15 (Y0), U?.2 (REG_A_LOW_OUT)
- new net: U?.18 (D4), U?.2 (A1)
- new net: U?.19 (D5), U?.3 (A2)
- new net: U?.16 (I_REG_ADDR_OUT), U?.7 (Y7)
- new net: U?.14 (I_REG_OPCODE_OUT), U?.9 (Y6)
- new net: U?.1 (S2), U?.46 (I1)
- new net: U?.10 (S4), U?.43 (I3)
- new net: U?.13 (S3), U?.44 (I2)
- new net: U?.4 (S1), U?.47 (I0)
- new net: U?.8 (GND), U?.9 (COUT)
- new net: U?.1 (S2), U?.40 (I5)
- new net: U?.10 (S4), U?.37 (I7)
- new net: U?.13 (S3), U?.38 (I6)
- new net: U?.4 (S1), U?.41 (I4)
- new net: U?.7 (CIN), U?.9 (COUT) (x2)
- new net: U?.1 (S2), U?.35 (I9)
- new net: U?.10 (S4), U?.32 (I11)
- new net: U?.13 (S3), U?.33 (I10)
- new net: U?.36 (I8), U?.4 (S1)
- new net: U?.1 (S2), U?.29 (I13)
- new net: U?.10 (S4), U?.26 (I15)
- new net: U?.13 (S3), U?.27 (I14)
- new net: U?.30 (I12), U?.4 (S1)
- new net: U?.26 (I15), U?.7 (Q7) (x2)
- new net: U?.27 (I14), U?.6 (Q6) (x2)
- new net: U?.29 (I13), U?.5 (Q5) (x2)
- new net: U?.30 (I12), U?.4 (Q4) (x2)
- new net: U?.3 (Q3), U?.32 (I11) (x2)
- new net: U?.2 (Q2), U?.33 (I10) (x2)
- new net: U?.1 (Q1), U?.35 (I9) (x2)
- new net: U?.15 (Q0), U?.36 (I8) (x2)
- new net +5V: U?.16 (VCC), U?.16 (VCC), U?.16 (VCC), U?.16 (VCC), U?.18 (Vcc), U?.18 (Vcc), U?.18 (Vcc), U?.18 (Vcc), U?.18 (Vcc), U?.18 (Vcc), U?.18 (Vcc), U?.18 (Vcc), U?.18 (Vcc), U?.18 (Vcc), U?.18 (Vcc), U?.18 (Vcc), U?.18 (Vcc), U?.18 (Vcc), U?.18 (Vcc), U?.18 (Vcc), U?.18 (Vcc), U?.18 (Vcc), U?.31 (Vcc), U?.31 (Vcc), U?.31 (Vcc), U?.31 (Vcc), U?.31 (Vcc), U?.31 (Vcc), U?.31 (Vcc), U?.31 (Vcc), U?.31 (Vcc), U?.31 (Vcc), U?.31 (Vcc), U?.31 (Vcc), U?.31 (Vcc), U?.31 (Vcc), U?.31 (Vcc), U?.31 (Vcc), U?.31 (Vcc), U?.31 (Vcc), U?.42 (Vcc), U?.42 (Vcc), U?.42 (Vcc), U?.42 (Vcc), U?.42 (Vcc), U?.42 (Vcc), U?.42 (Vcc), U?.42 (Vcc), U?.42 (Vcc), U?.42 (Vcc), U?.42 (Vcc), U?.42 (Vcc), U?.42 (Vcc), U?.42 (Vcc), U?.42 (Vcc), U?.42 (Vcc), U?.42 (Vcc), U?.42 (Vcc), U?.7 (Vcc), U?.7 (Vcc), U?.7 (Vcc), U?.7 (Vcc), U?.7 (Vcc), U?.7 (Vcc), U?.7 (Vcc), U?.7 (Vcc), U?.7 (Vcc), U?.7 (Vcc), U?.7 (Vcc), U?.7 (Vcc), U?.7 (Vcc), U?.7 (Vcc), U?.7 (Vcc), U?.7 (Vcc), U?.7 (Vcc), U?.7 (Vcc)
- new net A_HIGH_IN: U?.24 (OE4), U?.24 (OE4), U?.25 (OE3), U?.25 (OE3)
- new net A_HIGH_OUT: U?.19 (2Q4), U?.19 (2Q4), U?.24 (2OE), U?.24 (2OE)
- new net A_LOW_IN: U?.48 (OE2)
- new net Addr_BUS0: U?.2 (1Q0), U?.2 (1Q0)
- new net Addr_BUS1: U?.3 (1Q1), U?.3 (1Q1)
- new net Addr_BUS10: U?.16 (2Q2), U?.16 (2Q2)
- new net Addr_BUS11: U?.17 (2Q3), U?.17 (2Q3)
- new net Addr_BUS13: U?.20 (2Q5), U?.20 (2Q5)
- new net Addr_BUS14: U?.1 (1OE), U?.1 (1OE), U?.1 (1OE), U?.22 (2Q6), U?.22 (2Q6)
- new net Addr_BUS15: U?.23 (2Q7), U?.23 (2Q7)
- new net Addr_BUS2: U?.5 (1Q2), U?.5 (1Q2)
- new net Addr_BUS3: U?.6 (1Q3), U?.6 (1Q3)
- new net Addr_BUS4: U?.8 (1Q4), U?.8 (1Q4)
- new net Addr_BUS5: U?.9 (1Q5), U?.9 (1Q5)
- new net Addr_BUS6: U?.11 (1Q6), U?.11 (1Q6)
- new net Addr_BUS7: U?.12 (1Q7), U?.12 (1Q7)
- new net Addr_BUS8: U?.13 (2Q0), U?.13 (2Q0)
- new net Addr_BUS9: U?.14 (2Q1), U?.14 (2Q1)
- new net B_HIGH_IN: U?.24 (OE4), U?.24 (OE4), U?.24 (OE4), U?.24 (OE4), U?.25 (OE3), U?.25 (OE3), U?.25 (OE3), U?.25 (OE3)
- new net B_HIGH_OUT: U?.24 (2OE), U?.24 (2OE), U?.24 (2OE)
- new net B_LOW_IN: U?.1 (OE1), U?.1 (OE1), U?.1 (OE1), U?.48 (OE2), U?.48 (OE2), U?.48 (OE2)
- new net C_HIGH_IN: U?.24 (OE4), U?.25 (OE3)
- new net C_HIGH_OUT: U?.24 (2OE)
- new net Clock: U?.25 (2CP), U?.25 (2CP), U?.25 (2CP), U?.25 (2CP), U?.25 (2CP), U?.25 (2CP), U?.25 (2CP), U?.25 (2CP), U?.25 (2CP), U?.48 (1CP), U?.48 (1CP), U?.48 (1CP), U?.48 (1CP), U?.48 (1CP), U?.48 (1CP), U?.48 (1CP), U?.48 (1CP), U?.48 (1CP)
- new net D_HIGH_OUT: U?.24 (2OE)
- new net D_LOW_IN: U?.1 (OE1), U?.48 (OE2)
- new net D_LOW_OUT: U?.1 (1OE)
- new net Data_BUS0: U?.14 (2Q1), U?.14 (2Q1), U?.14 (2Q1), U?.14 (2Q1), U?.14 (2Q1), U?.14 (2Q1), U?.14 (2Q1), U?.14 (O9), U?.17 (2Q3), U?.17 (2Q3), U?.17 (2Q3), U?.17 (2Q3), U?.17 (2Q3), U?.17 (2Q3), U?.17 (2Q3), U?.17 (O11), U?.2 (1Q0), U?.2 (1Q0), U?.2 (1Q0), U?.2 (1Q0), U?.2 (1Q0), U?.2 (1Q0), U?.2 (1Q0), U?.2 (O0), U?.32 (I11), U?.32 (I11), U?.32 (I11), U?.32 (I11), U?.32 (I11), U?.32 (I11), U?.32 (I11), U?.35 (I9), U?.35 (I9), U?.35 (I9), U?.35 (I9), U?.35 (I9), U?.35 (I9), U?.35 (I9), U?.47 (I0), U?.47 (I0), U?.47 (I0), U?.47 (I0), U?.47 (I0), U?.47 (I0), U?.47 (I0)
- new net Data_BUS1: U?.13 (2Q0), U?.13 (2Q0), U?.13 (2Q0), U?.13 (2Q0), U?.13 (2Q0), U?.13 (2Q0), U?.13 (2Q0), U?.13 (O8), U?.16 (2Q2), U?.16 (2Q2), U?.16 (2Q2), U?.16 (2Q2), U?.16 (2Q2), U?.16 (2Q2), U?.16 (2Q2), U?.16 (O10), U?.3 (1Q1), U?.3 (1Q1), U?.3 (1Q1), U?.3 (1Q1), U?.3 (1Q1), U?.3 (1Q1), U?.3 (1Q1), U?.3 (O1), U?.33 (I10), U?.33 (I10), U?.33 (I10), U?.33 (I10), U?.33 (I10), U?.33 (I10), U?.33 (I10), U?.36 (I8), U?.36 (I8), U?.36 (I8), U?.36 (I8), U?.36 (I8), U?.36 (I8), U?.36 (I8), U?.46 (I1), U?.46 (I1), U?.46 (I1), U?.46 (I1), U?.46 (I1), U?.46 (I1), U?.46 (I1)
- new net Data_BUS12: U?.19 (2Q4), U?.19 (2Q4), U?.19 (2Q4), U?.19 (2Q4), U?.19 (2Q4), U?.19 (2Q4), U?.19 (2Q4), U?.19 (O12), U?.30 (I12), U?.30 (I12), U?.30 (I12), U?.30 (I12), U?.30 (I12), U?.30 (I12), U?.30 (I12)
- new net Data_BUS13: U?.20 (2Q5), U?.20 (2Q5), U?.20 (2Q5), U?.20 (2Q5), U?.20 (2Q5), U?.20 (2Q5), U?.20 (2Q5), U?.20 (O13), U?.29 (I13), U?.29 (I13), U?.29 (I13), U?.29 (I13), U?.29 (I13), U?.29 (I13), U?.29 (I13)
- new net Data_BUS14: U?.22 (2Q6), U?.22 (2Q6), U?.22 (2Q6), U?.22 (2Q6), U?.22 (2Q6), U?.22 (2Q6), U?.22 (2Q6), U?.22 (O14), U?.27 (I14), U?.27 (I14), U?.27 (I14), U?.27 (I14), U?.27 (I14), U?.27 (I14), U?.27 (I14)
- new net Data_BUS15: U?.23 (2Q7), U?.23 (2Q7), U?.23 (2Q7), U?.23 (2Q7), U?.23 (2Q7), U?.23 (2Q7), U?.23 (2Q7), U?.23 (O15), U?.26 (I15), U?.26 (I15), U?.26 (I15), U?.26 (I15), U?.26 (I15), U?.26 (I15), U?.26 (I15)
- new net Data_BUS2: U?.44 (I2), U?.44 (I2), U?.44 (I2), U?.44 (I2), U?.44 (I2), U?.44 (I2), U?.44 (I2), U?.5 (1Q2), U?.5 (1Q2), U?.5 (1Q2), U?.5 (1Q2), U?.5 (1Q2), U?.5 (1Q2), U?.5 (1Q2), U?.5 (O2)
- new net Data_BUS3: U?.43 (I3), U?.43 (I3), U?.43 (I3), U?.43 (I3), U?.43 (I3), U?.43 (I3), U?.43 (I3), U?.6 (1Q3), U?.6 (1Q3), U?.6 (1Q3), U?.6 (1Q3), U?.6 (1Q3), U?.6 (1Q3), U?.6 (1Q3), U?.6 (O3)
- new net Data_BUS4: U?.41 (I4), U?.41 (I4), U?.41 (I4), U?.41 (I4), U?.41 (I4), U?.41 (I4), U?.41 (I4), U?.8 (1Q4), U?.8 (1Q4), U?.8 (1Q4), U?.8 (1Q4), U?.8 (1Q4), U?.8 (1Q4), U?.8 (1Q4), U?.8 (O4)
- new net Data_BUS5: U?.40 (I5), U?.40 (I5), U?.40 (I5), U?.40 (I5), U?.40 (I5), U?.40 (I5), U?.40 (I5), U?.9 (1Q5), U?.9 (1Q5), U?.9 (1Q5), U?.9 (1Q5), U?.9 (1Q5), U?.9 (1Q5), U?.9 (1Q5), U?.9 (O5)
- new net Data_BUS6: U?.11 (1Q6), U?.11 (1Q6), U?.11 (1Q6), U?.11 (1Q6), U?.11 (1Q6), U?.11 (1Q6), U?.11 (1Q6), U?.11 (O6), U?.38 (I6), U?.38 (I6), U?.38 (I6), U?.38 (I6), U?.38 (I6), U?.38 (I6), U?.38 (I6)
- new net Data_BUS7: U?.12 (1Q7), U?.12 (1Q7), U?.12 (1Q7), U?.12 (1Q7), U?.12 (1Q7), U?.12 (1Q7), U?.12 (1Q7), U?.12 (O7), U?.37 (I7), U?.37 (I7), U?.37 (I7), U?.37 (I7), U?.37 (I7), U?.37 (I7), U?.37 (I7)
- new net E_HIGH_IN: U?.24 (OE4), U?.25 (OE3)
- new net E_HIGH_OUT: U?.24 (2OE)
- new net F_HIGH_IN: U?.24 (OE4), U?.25 (OE3)
- new net F_HIGH_OUT: U?.24 (2OE)
- new net F_LOW_IN: U?.1 (OE1), U?.48 (OE2)
- new net F_LOW_OUT: U?.1 (1OE)
- new net GND: U?.10 (GND), U?.10 (GND), U?.10 (GND), U?.10 (GND), U?.10 (GND), U?.10 (GND), U?.10 (GND), U?.10 (GND), U?.10 (GND), U?.10 (GND), U?.10 (GND), U?.10 (GND), U?.10 (GND), U?.10 (GND), U?.10 (GND), U?.10 (GND), U?.10 (GND), U?.10 (GND), U?.15 (GND), U?.15 (GND), U?.15 (GND), U?.15 (GND), U?.15 (GND), U?.15 (GND), U?.15 (GND), U?.15 (GND), U?.15 (GND), U?.15 (GND), U?.15 (GND), U?.15 (GND), U?.15 (GND), U?.15 (GND), U?.15 (GND), U?.15 (GND), U?.15 (GND), U?.15 (GND), U?.16 (GND), U?.16 (GND), U?.21 (GND), U?.21 (GND), U?.21 (GND), U?.21 (GND), U?.21 (GND), U?.21 (GND), U?.21 (GND), U?.21 (GND), U?.21 (GND), U?.21 (GND), U?.21 (GND), U?.21 (GND), U?.21 (GND), U?.21 (GND), U?.21 (GND), U?.21 (GND), U?.21 (GND), U?.21 (GND), U?.28 (GND), U?.28 (GND), U?.28 (GND), U?.28 (GND), U?.28 (GND), U?.28 (GND), U?.28 (GND), U?.28 (GND), U?.28 (GND), U?.28 (GND), U?.28 (GND), U?.28 (GND), U?.28 (GND), U?.28 (GND), U?.28 (GND), U?.28 (GND), U?.28 (GND), U?.28 (GND), U?.34 (GND), U?.34 (GND), U?.34 (GND), U?.34 (GND), U?.34 (GND), U?.34 (GND), U?.34 (GND), U?.34 (GND), U?.34 (GND), U?.34 (GND), U?.34 (GND), U?.34 (GND), U?.34 (GND), U?.34 (GND), U?.34 (GND), U?.34 (GND), U?.34 (GND), U?.34 (GND), U?.39 (GND), U?.39 (GND), U?.39 (GND), U?.39 (GND), U?.39 (GND), U?.39 (GND), U?.39 (GND), U?.39 (GND), U?.39 (GND), U?.39 (GND), U?.39 (GND), U?.39 (GND), U?.39 (GND), U?.39 (GND), U?.39 (GND), U?.39 (GND), U?.39 (GND), U?.39 (GND), U?.4 (GND), U?.4 (GND), U?.4 (GND), U?.4 (GND), U?.4 (GND), U?.4 (GND), U?.4 (GND), U?.4 (GND), U?.4 (GND), U?.4 (GND), U?.4 (GND), U?.4 (GND), U?.4 (GND), U?.4 (GND), U?.4 (GND), U?.4 (GND), U?.4 (GND), U?.4 (GND), U?.45 (GND), U?.45 (GND), U?.45 (GND), U?.45 (GND), U?.45 (GND), U?.45 (GND), U?.45 (GND), U?.45 (GND), U?.45 (GND), U?.45 (GND), U?.45 (GND), U?.45 (GND), U?.45 (GND), U?.45 (GND), U?.45 (GND), U?.45 (GND), U?.45 (GND), U?.45 (GND), U?.8 (GND), U?.8 (GND), U?.8 (GND)
- new net MAR_LOW: U?.1 (1OE)
- new net VCC: U?.32 (VCC), U?.32 (VCC)
Other:
- note added: "MAR\n"
- note added: "MDR"
- note added: "Register B\n"
- note added: "Register D\n"
- note added: "Register F\n"
- note removed: "CPU"
- note removed: "GPU"
- note removed: "Motherboard"
